File: pcb/pcb.kicad_pcb (KiCad board)
At the start: 2 copper layers, 132.5 x 101.5 mm, 46 parts

Commit message: fix: flipped underside RST/GND
Parts:
- moved _1 14.3 mm to (204.0, 109.7)
- moved D3 14.3 mm to (101.4, 84.9)
- moved D16 14.3 mm to (184.9, 130.8)
- moved D15 14.3 mm to (191.2, 69.2)
- moved H2 14.3 mm to (129.9, 128.7)
- moved H1 14.3 mm to (114.9, 82.6)
- moved S2 14.3 mm to (108.8, 107.7)
- moved PWR1 14.3 mm to (191.9, 62.3)
- moved D1 14.3 mm to (113.2, 121.0)
- moved D7 14.3 mm to (149.1, 92.0)
- moved S3 14.3 mm to (103.0, 89.6)
- moved MCU1 14.3 mm to (208.5, 115.7)
- moved S12 14.3 mm to (172.1, 69.1)
- moved S15 14.3 mm to (190.7, 74.1)
- moved S9 14.3 mm to (149.1, 58.9)
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Connections:
- MCU1 pad 17: GND2 -> RST
- MCU1 pad 18: RST -> GND2
- _3 pad 11: GND2 -> RST
- _4 pad 11: RST -> GND2
